Commit message: Cabo fixado ao drone e a um ponto fixo

File: src/pacote_do_drone/models/cabo.urdf (robot description, URDF)
Before this commit: robot cabo_flexivel, 71 links, 70 joints
Links:
- removed link dummy_1
- removed link dummy_10
- removed link dummy_11
- removed link dummy_12
- removed link dummy_13
- removed link dummy_14
- removed link dummy_15
- removed link dummy_16
- removed link dummy_17
- removed link dummy_18
- removed link dummy_19
- removed link dummy_2
- removed link dummy_20
- removed link dummy_21
- removed link dummy_22
- removed link dummy_23
- removed link dummy_24
- removed link dummy_25
- removed link dummy_26
- removed link dummy_27
- removed link dummy_28
- removed link dummy_29
- removed link dummy_3
- removed link dummy_30
- removed link dummy_31
- removed link dummy_32
- removed link dummy_33
- removed link dummy_34
- removed link dummy_35
- removed link dummy_4
- removed link dummy_5
- removed link dummy_6
- removed link dummy_7
- removed link dummy_8
- removed link dummy_9
- added link final_segment, mass 0.002; collision cylinder length=0.0425 radius=0.002; visual cylinder length=0.05 radius=0.002
- added link segment_36, mass 0.002; collision cylinder length=0.0425 radius=0.002; visual cylinder length=0.05 radius=0.002
- added link segment_37, mass 0.002; collision cylinder length=0.0425 radius=0.002; visual cylinder length=0.05 radius=0.002
- added link segment_38, mass 0.002; collision cylinder length=0.0425 radius=0.002; visual cylinder length=0.05 radius=0.002
- added link segment_39, mass 0.002; collision cylinder length=0.0425 radius=0.002; visual cylinder length=0.05 radius=0.002
- link raiz_cabo: mass 0.01 -> 0.02; geometry collision sphere 
- link segment_1: mass 0.001 -> 0.002; geometry collision cylinder length=0.0425 radius=0.002; visual cylinder length=0.05 radius=0.002
- link segment_10: mass 0.001 -> 0.002; geometry collision cylinder length=0.0425 radius=0.002; visual cylinder length=0.05 radius=0.002
- link segment_11: mass 0.001 -> 0.002; geometry collision cylinder length=0.0425 radius=0.002; visual cylinder length=0.05 radius=0.002
- link segment_12: mass 0.001 -> 0.002; geometry collision cylinder length=0.0425 radius=0.002; visual cylinder length=0.05 radius=0.002
- link segment_13: mass 0.001 -> 0.002; geometry collision cylinder length=0.0425 radius=0.002; visual cylinder length=0.05 radius=0.002
- link segment_14: mass 0.001 -> 0.002; geometry collision cylinder length=0.0425 radius=0.002; visual cylinder length=0.05 radius=0.002
- link segment_15: mass 0.001 -> 0.002; geometry collision cylinder length=0.0425 radius=0.002; visual cylinder length=0.05 radius=0.002
- link segment_16: mass 0.001 -> 0.002; geometry collision cylinder length=0.0425 radius=0.002; visual cylinder length=0.05 radius=0.002
- link segment_17: mass 0.001 -> 0.002; geometry collision cylinder length=0.0425 radius=0.002; visual cylinder length=0.05 radius=0.002
- link segment_18: mass 0.001 -> 0.002; geometry collision cylinder length=0.0425 radius=0.002; visual cylinder length=0.05 radius=0.002
- link segment_19: mass 0.001 -> 0.002; geometry collision cylinder length=0.0425 radius=0.002; visual cylinder length=0.05 radius=0.002
- link segment_2: mass 0.001 -> 0.002; geometry collision cylinder length=0.0425 radius=0.002; visual cylinder length=0.05 radius=0.002
- link segment_20: mass 0.001 -> 0.002; geometry collision cylinder length=0.0425 radius=0.002; visual cylinder length=0.05 radius=0.002
- link segment_21: mass 0.001 -> 0.002; geometry collision cylinder length=0.0425 radius=0.002; visual cylinder length=0.05 radius=0.002
- link segment_22: mass 0.001 -> 0.002; geometry collision cylinder length=0.0425 radius=0.002; visual cylinder length=0.05 radius=0.002
- link segment_23: mass 0.001 -> 0.002; geometry collision cylinder length=0.0425 radius=0.002; visual cylinder length=0.05 radius=0.002
- link segment_24: mass 0.001 -> 0.002; geometry collision cylinder length=0.0425 radius=0.002; visual cylinder length=0.05 radius=0.002
- link segment_25: mass 0.001 -> 0.002; geometry collision cylinder length=0.0425 radius=0.002; visual cylinder length=0.05 radius=0.002
- link segment_26: mass 0.001 -> 0.002; geometry collision cylinder length=0.0425 radius=0.002; visual cylinder length=0.05 radius=0.002
- link segment_27: mass 0.001 -> 0.002; geometry collision cylinder length=0.0425 radius=0.002; visual cylinder length=0.05 radius=0.002
- link segment_28: mass 0.001 -> 0.002; geometry collision cylinder length=0.0425 radius=0.002; visual cylinder length=0.05 radius=0.002
- link segment_29: mass 0.001 -> 0.002; geometry collision cylinder length=0.0425 radius=0.002; visual cylinder length=0.05 radius=0.002
- link segment_3: mass 0.001 -> 0.002; geometry collision cylinder length=0.0425 radius=0.002; visual cylinder length=0.05 radius=0.002
- link segment_30: mass 0.001 -> 0.002; geometry collision cylinder length=0.0425 radius=0.002; visual cylinder length=0.05 radius=0.002
- link segment_31: mass 0.001 -> 0.002; geometry collision cylinder length=0.0425 radius=0.002; visual cylinder length=0.05 radius=0.002
- link segment_32: mass 0.001 -> 0.002; geometry collision cylinder length=0.0425 radius=0.002; visual cylinder length=0.05 radius=0.002
- link segment_33: mass 0.001 -> 0.002; geometry collision cylinder length=0.0425 radius=0.002; visual cylinder length=0.05 radius=0.002
- link segment_34: mass 0.001 -> 0.002; geometry collision cylinder length=0.0425 radius=0.002; visual cylinder length=0.05 radius=0.002
- link segment_35: mass 0.001 -> 0.002; geometry collision cylinder length=0.0425 radius=0.002; visual cylinder length=0.05 radius=0.002
- link segment_4: mass 0.001 -> 0.002; geometry collision cylinder length=0.0425 radius=0.002; visual cylinder length=0.05 radius=0.002
- link segment_5: mass 0.001 -> 0.002; geometry collision cylinder length=0.0425 radius=0.002; visual cylinder length=0.05 radius=0.002
- link segment_6: mass 0.001 -> 0.002; geometry collision cylinder length=0.0425 radius=0.002; visual cylinder length=0.05 radius=0.002
- link segment_7: mass 0.001 -> 0.002; geometry collision cylinder length=0.0425 radius=0.002; visual cylinder length=0.05 radius=0.002
- link segment_8: mass 0.001 -> 0.002; geometry collision cylinder length=0.0425 radius=0.002; visual cylinder length=0.05 radius=0.002
- link segment_9: mass 0.001 -> 0.002; geometry collision cylinder length=0.0425 radius=0.002; visual cylinder length=0.05 radius=0.002
Joints:
- removed joint joint_10_x
- removed joint joint_10_y
- removed joint joint_11_x
- removed joint joint_11_y
- removed joint joint_12_x
- removed joint joint_12_y
- removed joint joint_13_x
- removed joint joint_13_y
- removed joint joint_14_x
- removed joint joint_14_y
- removed joint joint_15_x
- removed joint joint_15_y
- removed joint joint_16_x
- removed joint joint_16_y
- removed joint joint_17_x
- removed joint joint_17_y
- removed joint joint_18_x
- removed joint joint_18_y
- removed joint joint_19_x
- removed joint joint_19_y
- removed joint joint_1_x
- removed joint joint_1_y
- removed joint joint_20_x
- removed joint joint_20_y
- removed joint joint_21_x
- removed joint joint_21_y
- removed joint joint_22_x
- removed joint joint_22_y
- removed joint joint_23_x
- removed joint joint_23_y
- removed joint joint_24_x
- removed joint joint_24_y
- removed joint joint_25_x
- removed joint joint_25_y
- removed joint joint_26_x
- removed joint joint_26_y
- removed joint joint_27_x
- removed joint joint_27_y
- removed joint joint_28_x
- removed joint joint_28_y
- removed joint joint_29_x
- removed joint joint_29_y
- removed joint joint_2_x
- removed joint joint_2_y
- removed joint joint_30_x
- removed joint joint_30_y
- removed joint joint_31_x
- removed joint joint_31_y
- removed joint joint_32_x
- removed joint joint_32_y
- removed joint joint_33_x
- removed joint joint_33_y
- removed joint joint_34_x
- removed joint joint_34_y
- removed joint joint_35_x
- removed joint joint_35_y
- removed joint joint_3_x
- removed joint joint_3_y
- removed joint joint_4_x
- removed joint joint_4_y
- removed joint joint_5_x
- removed joint joint_5_y
- removed joint joint_6_x
- removed joint joint_6_y
- removed joint joint_7_x
- removed joint joint_7_y
- removed joint joint_8_x
- removed joint joint_8_y
- removed joint joint_9_x
- removed joint joint_9_y
- added joint joint_1: type revolute, parent raiz_cabo, child segment_1, origin xyz=0.0 0 0 rpy=0 -1.413716694115407 0, axis 0 1 0, limit lower=-2.0 upper=2.0 effort=5 velocity=10
- added joint joint_10: type revolute, parent segment_9, child segment_10, origin xyz=0.05 0 0 rpy=0 0.07068583470577035 0, axis 0 1 0, limit lower=-2.0 upper=2.0 effort=5 velocity=10
- added joint joint_11: type revolute, parent segment_10, child segment_11, origin xyz=0.05 0 0 rpy=0 0.07068583470577035 0, axis 0 1 0, limit lower=-2.0 upper=2.0 effort=5 velocity=10
- added joint joint_12: type revolute, parent segment_11, child segment_12, origin xyz=0.05 0 0 rpy=0 0.07068583470577035 0, axis 0 1 0, limit lower=-2.0 upper=2.0 effort=5 velocity=10
- added joint joint_13: type revolute, parent segment_12, child segment_13, origin xyz=0.05 0 0 rpy=0 0.07068583470577035 0, axis 0 1 0, limit lower=-2.0 upper=2.0 effort=5 velocity=10
- added joint joint_14: type revolute, parent segment_13, child segment_14, origin xyz=0.05 0 0 rpy=0 0.07068583470577035 0, axis 0 1 0, limit lower=-2.0 upper=2.0 effort=5 velocity=10
- added joint joint_15: type revolute, parent segment_14, child segment_15, origin xyz=0.05 0 0 rpy=0 0.07068583470577035 0, axis 0 1 0, limit lower=-2.0 upper=2.0 effort=5 velocity=10
- added joint joint_16: type revolute, parent segment_15, child segment_16, origin xyz=0.05 0 0 rpy=0 0.07068583470577035 0, axis 0 1 0, limit lower=-2.0 upper=2.0 effort=5 velocity=10
- added joint joint_17: type revolute, parent segment_16, child segment_17, origin xyz=0.05 0 0 rpy=0 0.07068583470577035 0, axis 0 1 0, limit lower=-2.0 upper=2.0 effort=5 velocity=10
- added joint joint_18: type revolute, parent segment_17, child segment_18, origin xyz=0.05 0 0 rpy=0 0.07068583470577035 0, axis 0 1 0, limit lower=-2.0 upper=2.0 effort=5 velocity=10
- added joint joint_19: type revolute, parent segment_18, child segment_19, origin xyz=0.05 0 0 rpy=0 0.07068583470577035 0, axis 0 1 0, limit lower=-2.0 upper=2.0 effort=5 velocity=10
- added joint joint_2: type revolute, parent segment_1, child segment_2, origin xyz=0.05 0 0 rpy=0 0.07068583470577035 0, axis 0 1 0, limit lower=-2.0 upper=2.0 effort=5 velocity=10
- added joint joint_20: type revolute, parent segment_19, child segment_20, origin xyz=0.05 0 0 rpy=0 0.07068583470577035 0, axis 0 1 0, limit lower=-2.0 upper=2.0 effort=5 velocity=10
- added joint joint_21: type revolute, parent segment_20, child segment_21, origin xyz=0.05 0 0 rpy=0 0.07068583470577035 0, axis 0 1 0, limit lower=-2.0 upper=2.0 effort=5 velocity=10
- added joint joint_22: type revolute, parent segment_21, child segment_22, origin xyz=0.05 0 0 rpy=0 0.07068583470577035 0, axis 0 1 0, limit lower=-2.0 upper=2.0 effort=5 velocity=10
- added joint joint_23: type revolute, parent segment_22, child segment_23, origin xyz=0.05 0 0 rpy=0 0.07068583470577035 0, axis 0 1 0, limit lower=-2.0 upper=2.0 effort=5 velocity=10
- added joint joint_24: type revolute, parent segment_23, child segment_24, origin xyz=0.05 0 0 rpy=0 0.07068583470577035 0, axis 0 1 0, limit lower=-2.0 upper=2.0 effort=5 velocity=10
- added joint joint_25: type revolute, parent segment_24, child segment_25, origin xyz=0.05 0 0 rpy=0 0.07068583470577035 0, axis 0 1 0, limit lower=-2.0 upper=2.0 effort=5 velocity=10
- added joint joint_26: type revolute, parent segment_25, child segment_26, origin xyz=0.05 0 0 rpy=0 0.07068583470577035 0, axis 0 1 0, limit lower=-2.0 upper=2.0 effort=5 velocity=10
- added joint joint_27: type revolute, parent segment_26, child segment_27, origin xyz=0.05 0 0 rpy=0 0.07068583470577035 0, axis 0 1 0, limit lower=-2.0 upper=2.0 effort=5 velocity=10
- added joint joint_28: type revolute, parent segment_27, child segment_28, origin xyz=0.05 0 0 rpy=0 0.07068583470577035 0, axis 0 1 0, limit lower=-2.0 upper=2.0 effort=5 velocity=10
- added joint joint_29: type revolute, parent segment_28, child segment_29, origin xyz=0.05 0 0 rpy=0 0.07068583470577035 0, axis 0 1 0, limit lower=-2.0 upper=2.0 effort=5 velocity=10
- added joint joint_3: type revolute, parent segment_2, child segment_3, origin xyz=0.05 0 0 rpy=0 0.07068583470577035 0, axis 0 1 0, limit lower=-2.0 upper=2.0 effort=5 velocity=10
- added joint joint_30: type revolute, parent segment_29, child segment_30, origin xyz=0.05 0 0 rpy=0 0.07068583470577035 0, axis 0 1 0, limit lower=-2.0 upper=2.0 effort=5 velocity=10
- added joint joint_31: type revolute, parent segment_30, child segment_31, origin xyz=0.05 0 0 rpy=0 0.07068583470577035 0, axis 0 1 0, limit lower=-2.0 upper=2.0 effort=5 velocity=10
- added joint joint_32: type revolute, parent segment_31, child segment_32, origin xyz=0.05 0 0 rpy=0 0.07068583470577035 0, axis 0 1 0, limit lower=-2.0 upper=2.0 effort=5 velocity=10
- added joint joint_33: type revolute, parent segment_32, child segment_33, origin xyz=0.05 0 0 rpy=0 0.07068583470577035 0, axis 0 1 0, limit lower=-2.0 upper=2.0 effort=5 velocity=10
- added joint joint_34: type revolute, parent segment_33, child segment_34, origin xyz=0.05 0 0 rpy=0 0.07068583470577035 0, axis 0 1 0, limit lower=-2.0 upper=2.0 effort=5 velocity=10
- added joint joint_35: type revolute, parent segment_34, child segment_35, origin xyz=0.05 0 0 rpy=0 0.07068583470577035 0, axis 0 1 0, limit lower=-2.0 upper=2.0 effort=5 velocity=10
- added joint joint_36: type revolute, parent segment_35, child segment_36, origin xyz=0.05 0 0 rpy=0 0.07068583470577035 0, axis 0 1 0, limit lower=-2.0 upper=2.0 effort=5 velocity=10
- added joint joint_37: type revolute, parent segment_36, child segment_37, origin xyz=0.05 0 0 rpy=0 0.07068583470577035 0, axis 0 1 0, limit lower=-2.0 upper=2.0 effort=5 velocity=10
- added joint joint_38: type revolute, parent segment_37, child segment_38, origin xyz=0.05 0 0 rpy=0 0.07068583470577035 0, axis 0 1 0, limit lower=-2.0 upper=2.0 effort=5 velocity=10
- added joint joint_39: type revolute, parent segment_38, child segment_39, origin xyz=0.05 0 0 rpy=0 0.07068583470577035 0, axis 0 1 0, limit lower=-2.0 upper=2.0 effort=5 velocity=10
- added joint joint_4: type revolute, parent segment_3, child segment_4, origin xyz=0.05 0 0 rpy=0 0.07068583470577035 0, axis 0 1 0, limit lower=-2.0 upper=2.0 effort=5 velocity=10
- added joint joint_40: type revolute, parent segment_39, child final_segment, origin xyz=0.05 0 0 rpy=0 0.07068583470577035 0, axis 0 1 0, limit lower=-2.0 upper=2.0 effort=5 velocity=10
- added joint joint_5: type revolute, parent segment_4, child segment_5, origin xyz=0.05 0 0 rpy=0 0.07068583470577035 0, axis 0 1 0, limit lower=-2.0 upper=2.0 effort=5 velocity=10
- added joint joint_6: type revolute, parent segment_5, child segment_6, origin xyz=0.05 0 0 rpy=0 0.07068583470577035 0, axis 0 1 0, limit lower=-2.0 upper=2.0 effort=5 velocity=10
- added joint joint_7: type revolute, parent segment_6, child segment_7, origin xyz=0.05 0 0 rpy=0 0.07068583470577035 0, axis 0 1 0, limit lower=-2.0 upper=2.0 effort=5 velocity=10
- added joint joint_8: type revolute, parent segment_7, child segment_8, origin xyz=0.05 0 0 rpy=0 0.07068583470577035 0, axis 0 1 0, limit lower=-2.0 upper=2.0 effort=5 velocity=10
- added joint joint_9: type revolute, parent segment_8, child segment_9, origin xyz=0.05 0 0 rpy=0 0.07068583470577035 0, axis 0 1 0, limit lower=-2.0 upper=2.0 effort=5 velocity=10

Commit message: Atulizações gerar_cabo.py

File: src/pacote_do_drone/models/cabo.urdf (robot description, URDF)
Before this commit: robot cabo_flexivel, 41 links, 40 joints
Links:
- added link ponta_cabo, mass 0.001
- link final_segment: mass 0.002 -> 0.0005
- link segment_1: mass 0.002 -> 0.0005
- link segment_10: mass 0.002 -> 0.0005
- link segment_11: mass 0.002 -> 0.0005
- link segment_12: mass 0.002 -> 0.0005
- link segment_13: mass 0.002 -> 0.0005
- link segment_14: mass 0.002 -> 0.0005
- link segment_15: mass 0.002 -> 0.0005
- link segment_16: mass 0.002 -> 0.0005
- link segment_17: mass 0.002 -> 0.0005
- link segment_18: mass 0.002 -> 0.0005
- link segment_19: mass 0.002 -> 0.0005
- link segment_2: mass 0.002 -> 0.0005
- link segment_20: mass 0.002 -> 0.0005
- link segment_21: mass 0.002 -> 0.0005
- link segment_22: mass 0.002 -> 0.0005
- link segment_23: mass 0.002 -> 0.0005
- link segment_24: mass 0.002 -> 0.0005
- link segment_25: mass 0.002 -> 0.0005
- link segment_26: mass 0.002 -> 0.0005
- link segment_27: mass 0.002 -> 0.0005
- link segment_28: mass 0.002 -> 0.0005
- link segment_29: mass 0.002 -> 0.0005
- link segment_3: mass 0.002 -> 0.0005
- link segment_30: mass 0.002 -> 0.0005
- link segment_31: mass 0.002 -> 0.0005
- link segment_32: mass 0.002 -> 0.0005
- link segment_33: mass 0.002 -> 0.0005
- link segment_34: mass 0.002 -> 0.0005
- link segment_35: mass 0.002 -> 0.0005
- link segment_36: mass 0.002 -> 0.0005
- link segment_37: mass 0.002 -> 0.0005
- link segment_38: mass 0.002 -> 0.0005
- link segment_39: mass 0.002 -> 0.0005
- link segment_4: mass 0.002 -> 0.0005
- link segment_5: mass 0.002 -> 0.0005
- link segment_6: mass 0.002 -> 0.0005
- link segment_7: mass 0.002 -> 0.0005
- link segment_8: mass 0.002 -> 0.0005
- link segment_9: mass 0.002 -> 0.0005
Joints:
- added joint joint_ponta: type fixed, parent final_segment, child ponta_cabo, origin xyz=0.05 0 0 rpy=0 0 0
- joint joint_1: origin xyz=0.0 0 0 rpy=0 -1.413716694115407 0 -> xyz=0.0 0 0 rpy=0 -2.036227962580655 0; type revolute -> ball
- joint joint_10: type revolute -> ball
- joint joint_11: type revolute -> ball
- joint joint_12: type revolute -> ball
- joint joint_13: type revolute -> ball
- joint joint_14: type revolute -> ball
- joint joint_15: type revolute -> ball
- joint joint_16: type revolute -> ball
- joint joint_17: type revolute -> ball
- joint joint_18: type revolute -> ball
- joint joint_19: type revolute -> ball
- joint joint_2: type revolute -> ball
- joint joint_20: type revolute -> ball
- joint joint_21: type revolute -> ball
- joint joint_22: type revolute -> ball
- joint joint_23: type revolute -> ball
- joint joint_24: type revolute -> ball
- joint joint_25: type revolute -> ball
- joint joint_26: type revolute -> ball
- joint joint_27: type revolute -> ball
- joint joint_28: type revolute -> ball
- joint joint_29: type revolute -> ball
- joint joint_3: type revolute -> ball
- joint joint_30: type revolute -> ball
- joint joint_31: type revolute -> ball
- joint joint_32: type revolute -> ball
- joint joint_33: type revolute -> ball
- joint joint_34: type revolute -> ball
- joint joint_35: type revolute -> ball
- joint joint_36: type revolute -> ball
- joint joint_37: type revolute -> ball
- joint joint_38: type revolute -> ball
- joint joint_39: type revolute -> ball
- joint joint_4: type revolute -> ball
- joint joint_40: type revolute -> ball
- joint joint_5: type revolute -> ball
- joint joint_6: type revolute -> ball
- joint joint_7: type revolute -> ball
- joint joint_8: type revolute -> ball
- joint joint_9: type revolute -> ball
